File: Soleac.kicad_sch (KiCad schematic)
At the start: 32 parts, among them J1 Regulador de voltaje, J2 Sensor MQ-2, SW1 SW_SPST, U1 LM358, U2 LM358, U3 ESP32-DEVKITC-32D, U4 ER_OLEDM0.91_1x-I2C

Commit message: Conexión Completa
Connections:
- net 3.3V: no longer U4.2 (VCC)
- net 5V: now also U4.2 (VCC)
Changed lines of the file:
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@@
 		)
 	)
-	(label "3.3V"
+	(label "5V"
 		(at 179.07 116.84 90)
 		(effects
