File: Hardware/Circuitos/Placa Mems - SOLEAC/Placa Mems - SOLEAC.kicad_pcb (KiCad board)
At the start: 2 copper layers, 50 x 50 mm, 7 parts, among them J2 Conn_01x04, J6 Conn_01x02, Y1 MA40S4R

Commit message: Placa Mems- Colocar plug ethernet
Parts:
- removed J2: Conn_01x04, Connector_RJ:RJ45_Amphenol_54602-x08_Horizontal
- added J1: Conn_01x08, Connector_RJ:RJ45_Amphenol_54602-x08_Horizontal, F.Cu at (46.1, 56.5)
- moved J6 3.30 mm to (49.3, 29.4)
Connections:
- net /GPIO39 c renamed /GPIO39 C
Routing:
- net /3.3V: track 100.8 -> 94.4 mm
- net /GPIO39 C: track 38.6 -> 33.0 mm
- net /entrada placa procesadora: track 10.8 -> 14.2 mm
- net /GPIO38 D: track 69.1 -> 67.8 mm
- added copper zone on F.Cu, net Earth
