File: Hardware/Circuitos/Sensor de gas MQ-9/Sensor de gas MQ-9.kicad_pcb (KiCad board)
At the start: 2 copper layers, 5 parts, among them J1 Conn_01x04, J2 Conn_01x02, J3 Conn_01x01

Commit message: Placa MQ9 - Colocación de componentes
Parts:
- J2: footprint Connector_PinHeader_2.54mm:PinHeader_1x02_P2.54mm_Vertical -> Connector_Molex:Molex_KK-254_AE-6410-02A_1x02_P2.54mm_Vertical
- R1, R2: footprint Resistor_THT:R_Axial_DIN0411_L9.9mm_D3.6mm_P15.24mm_Horizontal -> Resistor_THT:R_Axial_DIN0207_L6.3mm_D2.5mm_P7.62mm_Horizontal
- moved J2 61.4 mm to (124.8, 62.1), turned to 90 degrees
- moved R2 54.5 mm to (118.4, 67.4), turned to -90 degrees
- moved J1 53.3 mm to (112.2, 52.6), turned to 90 degrees
- moved R1 48.4 mm to (112.2, 59.8), turned to -90 degrees
- moved J3 43.8 mm to (112.2, 73.8), turned to -90 degrees
Other:
- board outline added: 25 x 30 mm

Commit message: Placa MQ9 - Ruteo PCB
Routing:
- net Net-(J3-Pin_1): track 0.00 -> 12.6 mm
- net Net-(J1-Pin_4): track 0.00 -> 9.00 mm
- net Net-(J1-Pin_1): track 0.00 -> 7.19 mm
- added copper zone on B.Cu, net Earth
Changed lines of the file:
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@@
 		(layer "Edge.Cuts")
+	)
+	(segment
+		(start 112.19 59.78)
+		(end 112.2 59.79)
+		(width 1)
+		(layer "B.Cu")
+		(net "Net-(J1-Pin_1)")
+	)
+	(segment
+		(start 112.19 52.6)
+		(end 112.19 59.78)
+		(width 1)
+		(layer "B.Cu")
+		(net "Net-(J1-Pin_1)")
+	)
+	(segment
+		(start 124.8 57.59)
+		(end 119.81 52.6)
+		(width 1)
+		(layer "B.Cu")
+		(net "Net-(J1-Pin_4)")
+	)
+	(segment
+		(start 124.8 59.535)
+		(end 124.8 57.59)
+		(width 1)
+		(layer "B.Cu")
+		(net "Net-(J1-Pin_4)")
+	)
+	(segment
+		(start 118.38 67.41)
+		(end 118.4 67.39)
+		(width 1)
+		(layer "B.Cu")
+		(net "Net-(J3-Pin_1)")
+	)
+	(segment
+		(start 112.2 67.41)
+		(end 112.2 73.8)
+		(width 1)
+		(layer "B.Cu")
+		(net "Net-(J3-Pin_1)")
+	)
+	(segment
+		(start 112.2 67.41)
+		(end 118.38 67.41)
+		(width 1)
+		(layer "B.Cu")
+		(net "Net-(J3-Pin_1)")
+	)
+	(zone
+		(net "Earth")
+		(layer "B.Cu")
+		(hatch edge 0.5)
+		(connect_pads
+			(clearance 0.5)
+		)
+		(min_thickness 0.25)
+		(fill yes
+			(thermal_gap 0.5)
+			(thermal_bridge_width 0.5)
+			(island_removal_mode 0)
+		)
+		(polygon
+			(pts
+				(xy 132 48.4) (xy 107 48.4) (xy 107 78.4) (xy 132 78.4)
+			)
+		)
 	)
 	(embedded_fonts no)
