File: Hardware/Circuitos/Placa Esp32S3/Placa ESP32.kicad_pcb (KiCad board)
At the start: 2 copper layers, 45 x 50 mm, 9 parts, among them J1 Conn_01x04, J3 ESP32-S3-Touch-LCD-3.5B, J4 Conn_01x02, J8 Conn_01x02

Commit message: Placa ESP32 - Cambio de huella bornera
Other:
- board size 45 x 50 mm -> 50 x 50 mm
Changed lines of the file:
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@@
 	(gr_rect
 		(start 69.6 75.4)
-		(end 114.6 125.4)
+		(end 119.6 125.4)
 		(stroke
 			(width 0.05)
@@
 	)
 	(segment
+		(start 104.6 110.55)
+		(end 101.07 107.02)
+		(width 1.5)
+		(layer "F.Cu")
+		(net "/GPIO10 (Entrada Murata)")
+	)
+	(segment
+		(start 102.2 103.21)
+		(end 102.2 105.89)
+		(width 1.5)
+		(layer "F.Cu")
+		(net "/GPIO10 (Entrada Murata)")
+	)
+	(segment
+		(start 90.82 107)
+		(end 90.8 107.02)
+		(width 1.5)
+		(layer "F.Cu")
+		(net "/GPIO10 (Entrada Murata)")
+	)
+	(segment
+		(start 101.07 107.02)
+		(end 90.8 107.02)
+		(width 1.5)
+		(layer "F.Cu")
+		(net "/GPIO10 (Entrada Murata)")
+	)
+	(segment
+		(start 107 98.99)
+		(end 106.42 98.99)
+		(width 1.5)
+		(layer "F.Cu")
+		(net "/GPIO10 (Entrada Murata)")
+	)
+	(segment
+		(start 106.42 98.99)
+		(end 102.2 103.21)
+		(width 1.5)
+		(layer "F.Cu")
+		(net "/GPIO10 (Entrada Murata)")
+	)
+	(segment
+		(start 102.2 105.89)
+		(end 101.07 107.02)
+		(width 1.5)
+		(layer "F.Cu")
+		(net "/GPIO10 (Entrada Murata)")
+	)
+	(segment
 		(start 103.35 94.44)
 		(end 102.2 95.59)
@@
 	)
 	(segment
+		(start 97 85.6)
+		(end 93.02 81.62)
+		(width 1.5)
+		(layer "F.Cu")
+		(net "/3.3V")
+	)
+	(segment
+		(start 90.8 79)
+		(end 90.2 78.4)
+		(width 1.5)
+		(layer "F.Cu")
+		(net "/3.3V")
+	)
+	(segment
+		(start 90.8 81.62)
+		(end 90.8 79)
+		(width 1.5)
+		(layer "F.Cu")
+		(net "/3.3V")
+	)
+	(segment
+		(start 73.61 109.41)
+		(end 77.02 109.41)
+		(width 1.5)
+		(layer "F.Cu")
+		(net "/3.3V")
+	)
+	(segment
+		(start 93.02 81.62)
+		(end 90.8 81.62)
+		(width 1.5)
+		(layer "F.Cu")
+		(net "/3.3V")
+	)
+	(segment
+		(start 90.2 78.4)
+		(end 83.4 78.4)
+		(width 1.5)
+		(layer "F.Cu")
+		(net "/3.3V")
+	)
+	(segment
+		(start 72 89.8)
+		(end 72 107.8)
+		(width 1.5)
+		(layer "F.Cu")
+		(net "/3.3V")
+	)
+	(segment
+		(start 97 103.39)
+		(end 97 85.6)
+		(width 1.5)
+		(layer "F.Cu")
+		(net "/3.3V")
+	)
+	(segment
+		(start 83.4 78.4)
+		(end 72 89.8)
+		(width 1.5)
+		(layer "F.Cu")
+		(net "/3.3V")
+	)
+	(segment
+		(start 72 107.8)
+		(end 73.61 109.41)
+		(width 1.5)
+		(layer "F.Cu")
+		(net "/3.3V")
+	)
+	(segment
+		(start 77.02 106.87)
+		(end 88.16 106.87)
+		(width 1.5)
+		(layer "F.Cu")
+		(net "/GPIO40")
+	)
+	(segment
+		(start 88.16 106.87)
+		(end 88.3 107.01)
+		(width 1.5)
+		(layer "F.Cu")
+		(net "/GPIO40")
+	)
+	(segment
+		(start 88.3 104.47)
+		(end 77.16 104.47)
+		(width 1.5)
+		(layer "F.Cu")
+		(net "/GPIO41")
+	)
+	(segment
+		(start 77.16 104.47)
+		(end 77.02 104.33)
+		(width 1.5)
+		(layer "F.Cu")
+		(net "/GPIO41")
+	)
+	(segment
 		(start 110.6 117.8)
 		(end 107.2 121.2)
@@
 	)
 	(segment
-		(start 77.02 106.87)
-		(end 88.16 106.87)
-		(width 1.5)
-		(layer "F.Cu")
-		(net "/GPIO40")
-	)
-	(segment
-		(start 88.16 106.87)
-		(end 88.3 107.01)
-		(width 1.5)
-		(layer "F.Cu")
-		(net "/GPIO40")
-	)
-	(segment
-		(start 88.3 104.47)
-		(end 77.16 104.47)
-		(width 1.5)
-		(layer "F.Cu")
-		(net "/GPIO41")
-	)
-	(segment
-		(start 77.16 104.47)
-		(end 77.02 104.33)
-		(width 1.5)
-		(layer "F.Cu")
-		(net "/GPIO41")
-	)
-	(segment
-		(start 97 85.6)
-		(end 93.02 81.62)
-		(width 1.5)
-		(layer "F.Cu")
-		(net "/3.3V")
-	)
-	(segment
-		(start 90.8 79)
-		(end 90.2 78.4)
-		(width 1.5)
-		(layer "F.Cu")
-		(net "/3.3V")
-	)
-	(segment
-		(start 90.8 81.62)
-		(end 90.8 79)
-		(width 1.5)
-		(layer "F.Cu")
-		(net "/3.3V")
-	)
-	(segment
-		(start 73.61 109.41)
-		(end 77.02 109.41)
-		(width 1.5)
-		(layer "F.Cu")
-		(net "/3.3V")
-	)
-	(segment
-		(start 93.02 81.62)
-		(end 90.8 81.62)
-		(width 1.5)
-		(layer "F.Cu")
-		(net "/3.3V")
-	)
-	(segment
-		(start 90.2 78.4)
-		(end 83.4 78.4)
-		(width 1.5)
-		(layer "F.Cu")
-		(net "/3.3V")
-	)
-	(segment
-		(start 72 89.8)
-		(end 72 107.8)
-		(width 1.5)
-		(layer "F.Cu")
-		(net "/3.3V")
-	)
-	(segment
-		(start 97 103.39)
-		(end 97 85.6)
-		(width 1.5)
-		(layer "F.Cu")
-		(net "/3.3V")
-	)
-	(segment
-		(start 83.4 78.4)
-		(end 72 89.8)
-		(width 1.5)
-		(layer "F.Cu")
-		(net "/3.3V")
-	)
-	(segment
-		(start 72 107.8)
-		(end 73.61 109.41)
-		(width 1.5)
-		(layer "F.Cu")
-		(net "/3.3V")
-	)
-	(segment
 		(start 96.99 117.4)
 		(end 96.99 111.02)
@@
 		(layer "F.Cu")
 		(net "Net-(D6-A)")
-	)
-	(segment
-		(start 104.6 110.55)
-		(end 101.07 107.02)
-		(width 1.5)
-		(layer "F.Cu")
-		(net "/GPIO10 (Entrada Murata)")
-	)
-	(segment
-		(start 102.2 103.21)
-		(end 102.2 105.89)
-		(width 1.5)
-		(layer "F.Cu")
-		(net "/GPIO10 (Entrada Murata)")
-	)
-	(segment
-		(start 90.82 107)
-		(end 90.8 107.02)
-		(width 1.5)
-		(layer "F.Cu")
-		(net "/GPIO10 (Entrada Murata)")
-	)
-	(segment
-		(start 101.07 107.02)
-		(end 90.8 107.02)
-		(width 1.5)
-		(layer "F.Cu")
-		(net "/GPIO10 (Entrada Murata)")
-	)
-	(segment
-		(start 107 98.99)
-		(end 106.42 98.99)
-		(width 1.5)
-		(layer "F.Cu")
-		(net "/GPIO10 (Entrada Murata)")
-	)
-	(segment
-		(start 106.42 98.99)
-		(end 102.2 103.21)
-		(width 1.5)
-		(layer "F.Cu")
-		(net "/GPIO10 (Entrada Murata)")
-	)
-	(segment
-		(start 102.2 105.89)
-		(end 101.07 107.02)
-		(width 1.5)
-		(layer "F.Cu")
-		(net "/GPIO10 (Entrada Murata)")
 	)
 	(zone
@@
 		)
 		(min_thickness 0.25)
-		(fill yes
+		(fill
 			(thermal_gap 0.5)
 			(thermal_bridge_width 0.5)
@@
 		(polygon
 			(pts
-				(xy 114.6 125.4) (xy 69.6 125.4) (xy 69.6 75.4) (xy 114.6 75.4)
+				(xy 119.6 125.4) (xy 69.6 125.4) (xy 69.6 75.4) (xy 119.6 75.4)
 			)
 		)

Commit message: Placa ESP32 - Actualizar huella en PCB
Parts:
- J8: footprint Connector_Molex:Molex_KK-254_AE-6410-02A_1x02_P2.54mm_Vertical -> Connector_Molex:Molex_KK-254_AE-6410-04A_1x04_P2.54mm_Vertical
- moved J8 5.01 mm to (116.4, 80.6)
Routing:
- net /5V: track 59.9 -> 17.1 mm
Changed lines of the file:
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@@
 		)
 	)
-	(footprint "Connector_Molex:Molex_KK-254_AE-6410-02A_1x02_P2.54mm_Vertical"
-		(layer "F.Cu")
-		(at 111.390591 80.567277 180)
-		(descr "Molex KK-254 Interconnect System, old/engineering part number: AE-6410-02A example for new part number: 22-27-2021, 2 Pins (http://www.molex.com/pdm_docs/sd/022272021_sd.pdf)")
+	(footprint "Connector_Molex:Molex_KK-254_AE-6410-04A_1x04_P2.54mm_Vertical"
+		(layer "F.Cu")
+		(at 116.4 80.6 180)
+		(descr "Molex KK-254 Interconnect System, old/engineering part number: AE-6410-04A example for new part number: 22-27-2041, 4 Pins (http://www.molex.com/pdm_docs/sd/022272021_sd.pdf)")
 		(tags "connector Molex KK-254 vertical")
 		(property "Reference" "J8"
-			(at 1.27 -4.12 0)
+			(at 3.81 -4.12 180)
 			(layer "F.SilkS")
 			(effects
@@
 		)
 		(property "Value" "Conn_01x02"
-			(at 1.27 4.08 0)
+			(at 3.81 4.08 180)
 			(layer "F.Fab")
 			(effects
@@
 		)
 		(property "Datasheet" ""
-			(at 0 0 0)
+			(at 0 0 180)
 			(layer "F.Fab")
 			(hide yes)
@@
 		)
 		(property "Description" "Generic connector, single row, 01x02, script generated (kicad-library-utils/schlib/autogen/connector/)"
-			(at 0 0 0)
+			(at 0 0 180)
 			(layer "F.Fab")
 			(hide yes)
@@
 		)
 		(property "KiLib_Generator" "connector/Molex"
-			(at 0 0 0)
+			(at 0 0 180)
 			(layer "F.SilkS")
 			(hide yes)
@@
 		(duplicate_pad_numbers_are_jumpers no)
 		(fp_line
+			(start 8.42 -2.43)
+			(end 8.42 -3.03)
+			(stroke
+				(width 0.12)
+				(type solid)
+			)
+			(layer "F.SilkS")
+		)
+		(fp_line
+			(start 7.62 1.99)
+			(end 7.62 2.99)
+			(stroke
+				(width 0.12)
+				(type solid)
+			)
+			(layer "F.SilkS")
+		)
+		(fp_line
+			(start 7.37 2.99)
+			(end 7.37 1.99)
+			(stroke
+				(width 0.12)
+				(type solid)
+			)
+			(layer "F.SilkS")
+		)
+		(fp_line
+			(start 7.37 1.46)
+			(end 7.62 1.99)
+			(stroke
+				(width 0.12)
+				(type solid)
+			)
+			(layer "F.SilkS")
+		)
+		(fp_line
+			(start 6.82 -2.43)
+			(end 8.42 -2.43)
+			(stroke
+				(width 0.12)
+				(type solid)
+			)
+			(layer "F.SilkS")
+		)
+		(fp_line
+			(start 6.82 -3.03)
+			(end 6.82 -2.43)
+			(stroke
+				(width 0.12)
+				(type solid)
+			)
+			(layer "F.SilkS")
+		)
+		(fp_line
+			(start 5.88 -2.43)
+			(end 5.88 -3.03)
+			(stroke
+				(width 0.12)
+				(type solid)
+			)
+			(layer "F.SilkS")
+		)
+		(fp_line
+			(start 4.28 -2.43)
+			(end 5.88 -2.43)
+			(stroke
+				(width 0.12)
+				(type solid)
+			)
+			(layer "F.SilkS")
+		)
+		(fp_line
+			(start 4.28 -3.03)
+			(end 4.28 -2.43)
+			(stroke
+				(width 0.12)
+				(type solid)
+			)
+			(layer "F.SilkS")
+		)
+		(fp_line
 			(start 3.34 -2.43)
 			(end 3.34 -3.03)
@@
 		)
 		(fp_line
-			(start 2.54 1.99)
-			(end 2.54 2.99)
-			(stroke
-				(width 0.12)
-				(type solid)
-			)
-			(layer "F.SilkS")
-		)
-		(fp_line
-			(start 2.29 2.99)
-			(end 2.29 1.99)
-			(stroke
-				(width 0.12)
-				(type solid)
-			)
-			(layer "F.SilkS")
-		)
-		(fp_line
-			(start 2.29 1.46)
-			(end 2.54 1.99)
-			(stroke
-				(width 0.12)
-				(type solid)
-			)
-			(layer "F.SilkS")
-		)
-		(fp_line
 			(start 1.74 -2.43)
 			(end 3.34 -2.43)
@@
 		(fp_line
 			(start 0.25 1.46)
-			(end 2.29 1.46)
+			(end 7.37 1.46)
 			(stroke
 				(width 0.12)
@@
 		(fp_line
 			(start 0 1.99)
-			(end 2.54 1.99)
+			(end 7.62 1.99)
 			(stroke
 				(width 0.12)
@@
 		(fp_rect
 			(start -1.38 -3.03)
-			(end 3.92 2.99)
+			(end 9 2.99)
 			(stroke
 				(width 0.12)
@@
 		(fp_rect
 			(start -1.77 -3.42)
-			(end 4.32 3.38)
+			(end 9.39 3.38)
 			(stroke
 				(width 0.05)
@@
 		(fp_rect
 			(start -1.27 -2.92)
-			(end 3.81 2.88)
+			(end 8.89 2.88)
 			(stroke
 				(width 0.1)
@@
 		)
 		(fp_text user "${REFERENCE}"
-			(at 1.27 -2.22 0)
+			(at 3.81 -2.22 180)
 			(layer "F.Fab")
 			(effects
@@
 			(pintype "passive")
 		)
+		(pad "3" thru_hole oval
+			(at 5.08 0 180)
+			(size 1.74 2.19)
+			(drill 1.19)
+			(layers "*.Cu" "*.Mask")
+			(remove_unused_layers no)
+		)
+		(pad "4" thru_hole oval
+			(at 7.62 0 180)
+			(size 1.74 2.19)
+			(drill 1.19)
+			(layers "*.Cu" "*.Mask")
+			(remove_unused_layers no)
+		)
 		(embedded_fonts no)
-		(model "${KICAD10_3DMODEL_DIR}/Connector_Molex.3dshapes/Molex_KK-254_AE-6410-02A_1x02_P2.54mm_Vertical.step"
+		(model "${KICAD10_3DMODEL_DIR}/Connector_Molex.3dshapes/Molex_KK-254_AE-6410-04A_1x04_P2.54mm_Vertical.step"
 			(offset
 				(xyz 0 0 0)
@@
 	)
 	(segment
-		(start 110.6 117.8)
-		(end 107.2 121.2)
-		(width 1.5)
-		(layer "F.Cu")
-		(net "/5V")
-	)
-	(segment
-		(start 110.6 95.6)
-		(end 110.6 117.8)
-		(width 1.5)
-		(layer "F.Cu")
-		(net "/5V")
-	)
-	(segment
 		(start 108.935 80.58)
 		(end 108.863314 80.58)
@@
 	)
 	(segment
-		(start 108.850591 80.567277)
-		(end 108.850591 93.850591)
-		(width 1.5)
-		(layer "F.Cu")
-		(net "/5V")
-	)
-	(segment
 		(start 108.863314 80.58)
 		(end 108.850591 80.567277)
 		(width 1.5)
 		(layer "F.Cu")
-		(net "/5V")
-	)
-	(segment
-		(start 108.850591 93.850591)
-		(end 110.6 95.6)
-		(width 1.5)
-		(layer "F.Cu")

Commit message: Placa ESP - Actualizacion bornera
Parts:
- J8: footprint Connector_Molex:Molex_KK-254_AE-6410-04A_1x04_P2.54mm_Vertical -> Connector_Molex:Molex_KK-254_AE-6410-02A_1x02_P2.54mm_Vertical
- moved J8 13.8 mm to (114.4, 94.3), turned to 90 degrees
Routing:
- net /5V: track 17.1 -> 56.3 mm
Changed lines of the file:
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@@
 		)
 	)
-	(footprint "Connector_Molex:Molex_KK-254_AE-6410-04A_1x04_P2.54mm_Vertical"
-		(layer "F.Cu")
-		(at 116.4 80.6 180)
-		(descr "Molex KK-254 Interconnect System, old/engineering part number: AE-6410-04A example for new part number: 22-27-2041, 4 Pins (http://www.molex.com/pdm_docs/sd/022272021_sd.pdf)")
+	(footprint "Connector_Molex:Molex_KK-254_AE-6410-02A_1x02_P2.54mm_Vertical"
+		(layer "F.Cu")
+		(at 114.4 94.275 90)
+		(descr "Molex KK-254 Interconnect System, old/engineering part number: AE-6410-02A example for new part number: 22-27-2021, 2 Pins (http://www.molex.com/pdm_docs/sd/022272021_sd.pdf)")
 		(tags "connector Molex KK-254 vertical")
 		(property "Reference" "J8"
-			(at 3.81 -4.12 180)
+			(at 1.27 -4.12 90)
 			(layer "F.SilkS")
 			(effects
@@
 		)
 		(property "Value" "Conn_01x02"
-			(at 3.81 4.08 180)
+			(at 1.27 4.08 90)
 			(layer "F.Fab")
 			(effects
@@
 		)
 		(property "Datasheet" ""
-			(at 0 0 180)
+			(at 0 0 90)
 			(layer "F.Fab")
 			(hide yes)
@@
 		)
 		(property "Description" "Generic connector, single row, 01x02, script generated (kicad-library-utils/schlib/autogen/connector/)"
-			(at 0 0 180)
+			(at 0 0 90)
 			(layer "F.Fab")
 			(hide yes)
@@
 		)
 		(property "KiLib_Generator" "connector/Molex"
-			(at 0 0 180)
+			(at 0 0 90)
 			(layer "F.SilkS")
 			(hide yes)
@@
 		(duplicate_pad_numbers_are_jumpers no)
 		(fp_line
-			(start 8.42 -2.43)
-			(end 8.42 -3.03)
-			(stroke
-				(width 0.12)
-				(type solid)
-			)
-			(layer "F.SilkS")
-		)
-		(fp_line
-			(start 7.62 1.99)
-			(end 7.62 2.99)
-			(stroke
-				(width 0.12)
-				(type solid)
-			)
-			(layer "F.SilkS")
-		)
-		(fp_line
-			(start 7.37 2.99)
-			(end 7.37 1.99)
-			(stroke
-				(width 0.12)
-				(type solid)
-			)
-			(layer "F.SilkS")
-		)
-		(fp_line
-			(start 7.37 1.46)
-			(end 7.62 1.99)
-			(stroke
-				(width 0.12)
-				(type solid)
-			)
-			(layer "F.SilkS")
-		)
-		(fp_line
-			(start 6.82 -2.43)
-			(end 8.42 -2.43)
-			(stroke
-				(width 0.12)
-				(type solid)
-			)
-			(layer "F.SilkS")
-		)
-		(fp_line
-			(start 6.82 -3.03)
-			(end 6.82 -2.43)
-			(stroke
-				(width 0.12)
-				(type solid)
-			)
-			(layer "F.SilkS")
-		)
-		(fp_line
-			(start 5.88 -2.43)
-			(end 5.88 -3.03)
-			(stroke
-				(width 0.12)
-				(type solid)
-			)
-			(layer "F.SilkS")
-		)
-		(fp_line
-			(start 4.28 -2.43)
-			(end 5.88 -2.43)
-			(stroke
-				(width 0.12)
-				(type solid)
-			)
-			(layer "F.SilkS")
-		)
-		(fp_line
-			(start 4.28 -3.03)
-			(end 4.28 -2.43)
+			(start 1.74 -3.03)
+			(end 1.74 -2.43)
+			(stroke
+				(width 0.12)
+				(type solid)
+			)
+			(layer "F.SilkS")
+		)
+		(fp_line
+			(start -0.8 -3.03)
+			(end -0.8 -2.43)
 			(stroke
 				(width 0.12)
@@
 		)
 		(fp_line
-			(start 1.74 -3.03)
-			(end 1.74 -2.43)
-			(stroke
-				(width 0.12)
-				(type solid)
-			)
-			(layer "F.SilkS")
-		)
-		(fp_line
 			(start 0.8 -2.43)
 			(end 0.8 -3.03)
@@
 		)
 		(fp_line
+			(start -0.8 -2.43)
+			(end 0.8 -2.43)
+			(stroke
+				(width 0.12)
+				(type solid)
+			)
+			(layer "F.SilkS")
+		)
+		(fp_line
+			(start -1.67 -2)
+			(end -1.67 2)
+			(stroke
+				(width 0.12)
+				(type solid)
+			)
+			(layer "F.SilkS")
+		)
+		(fp_line
+			(start 2.29 1.46)
+			(end 2.54 1.99)
+			(stroke
+				(width 0.12)
+				(type solid)
+			)
+			(layer "F.SilkS")
+		)
+		(fp_line
+			(start 0.25 1.46)
+			(end 2.29 1.46)
+			(stroke
+				(width 0.12)
+				(type solid)
+			)
+			(layer "F.SilkS")
+		)
+		(fp_line
+			(start 2.54 1.99)
+			(end 2.54 2.99)
+			(stroke
+				(width 0.12)
+				(type solid)
+			)
+			(layer "F.SilkS")
+		)
+		(fp_line
+			(start 0 1.99)
+			(end 0.25 1.46)
+			(stroke
+				(width 0.12)
+				(type solid)
+			)
+			(layer "F.SilkS")
+		)
+		(fp_line
+			(start 0 1.99)
+			(end 2.54 1.99)
+			(stroke
+				(width 0.12)
+				(type solid)
+			)
+			(layer "F.SilkS")
+		)
+		(fp_line
+			(start 2.29 2.99)
+			(end 2.29 1.99)
+			(stroke
+				(width 0.12)
+				(type solid)
+			)
+			(layer "F.SilkS")
+		)
+		(fp_line
 			(start 0.25 2.99)
 			(end 0.25 1.99)
@@
 		)
 		(fp_line
-			(start 0.25 1.46)
-			(end 7.37 1.46)
-			(stroke
-				(width 0.12)
-				(type solid)
-			)
-			(layer "F.SilkS")
-		)
-		(fp_line
 			(start 0 2.99)
 			(end 0 1.99)
@@
 			(layer "F.SilkS")
 		)
-		(fp_line
-			(start 0 1.99)
-			(end 7.62 1.99)
-			(stroke
-				(width 0.12)
-				(type solid)
-			)
-			(layer "F.SilkS")
-		)
-		(fp_line
-			(start 0 1.99)
-			(end 0.25 1.46)
-			(stroke
-				(width 0.12)
-				(type solid)
-			)
-			(layer "F.SilkS")
-		)
-		(fp_line
-			(start -0.8 -2.43)
-			(end 0.8 -2.43)
-			(stroke
-				(width 0.12)
-				(type solid)
-			)
-			(layer "F.SilkS")
-		)
-		(fp_line
-			(start -0.8 -3.03)
-			(end -0.8 -2.43)
-			(stroke
-				(width 0.12)
-				(type solid)
-			)
-			(layer "F.SilkS")
-		)
-		(fp_line
-			(start -1.67 -2)
-			(end -1.67 2)
-			(stroke
-				(width 0.12)
-				(type solid)
-			)
-			(layer "F.SilkS")
-		)
 		(fp_rect
 			(start -1.38 -3.03)
-			(end 9 2.99)
+			(end 3.92 2.99)
 			(stroke
 				(width 0.12)
@@
 		(fp_rect
 			(start -1.77 -3.42)
-			(end 9.39 3.38)
+			(end 4.32 3.38)
 			(stroke
 				(width 0.05)
@@
 		)
 		(fp_line
+			(start -1.27 -0.5)
+			(end -0.562893 0)
+			(stroke
+				(width 0.1)
+				(type solid)
+			)
+			(layer "F.Fab")
+		)
+		(fp_line
 			(start -0.562893 0)
 			(end -1.27 0.5)
@@
 			(layer "F.Fab")
 		)
-		(fp_line
-			(start -1.27 -0.5)
-			(end -0.562893 0)
-			(stroke
-				(width 0.1)
-				(type solid)
-			)
-			(layer "F.Fab")
-		)
 		(fp_rect
 			(start -1.27 -2.92)
-			(end 8.89 2.88)
+			(end 3.81 2.88)
 			(stroke
 				(width 0.1)
@@
 		)
 		(fp_text user "${REFERENCE}"
-			(at 3.81 -2.22 180)
+			(at 1.27 -2.22 90)
 			(layer "F.Fab")
 			(effects
@@
 		)
 		(pad "1" thru_hole roundrect
-			(at 0 0 180)
+			(at 0 0 90)
 			(size 1.74 2.19)
 			(drill 1.19)
@@
 		)
 		(pad "2" thru_hole oval
-			(at 2.54 0 180)
+			(at 2.54 0 90)
 			(size 1.74 2.19)
 			(drill 1.19)
@@
 			(pintype "passive")
 		)
-		(pad "3" thru_hole oval
-			(at 5.08 0 180)
-			(size 1.74 2.19)
-			(drill 1.19)
-			(layers "*.Cu" "*.Mask")
-			(remove_unused_layers no)
-		)
-		(pad "4" thru_hole oval
-			(at 7.62 0 180)
-			(size 1.74 2.19)
-			(drill 1.19)
-			(layers "*.Cu" "*.Mask")
-			(remove_unused_layers no)
-		)
 		(embedded_fonts no)
-		(model "${KICAD10_3DMODEL_DIR}/Connector_Molex.3dshapes/Molex_KK-254_AE-6410-04A_1x04_P2.54mm_Vertical.step"
+		(model "${KICAD10_3DMODEL_DIR}/Connector_Molex.3dshapes/Molex_KK-254_AE-6410-02A_1x02_P2.54mm_Vertical.step"
 			(offset
 				(xyz 0 0 0)
@@
 	)
 	(segment
-		(start 108.935 80.58)
-		(end 108.863314 80.58)
+		(start 116 118.2)
+		(end 116 100)
 		(width 1.5)
 		(layer "F.Cu")
@@
 	)
 	(segment
-		(start 107.2 121.2)
+		(start 90.8 119.72)
 		(end 92.28 121.2)
 		(width 1.5)
@@
 	(segment
 		(start 92.28 121.2)
-		(end 90.8 119.72)
+		(end 113 121.2)
 		(width 1.5)
 		(layer "F.Cu")
@@
 	)
 	(segment
-		(start 108.863314 80.58)
-		(end 108.850591 80.567277)
+		(start 116.048984 91.735)
+		(end 114.4 91.735)
+		(width 1.5)
+		(layer "F.Cu")
+		(net "/5V")
+	)
+	(segment
+		(start 117.4 93.086016)
+		(end 116.048984 91.735)
+		(width 1.5)
+		(layer "F.Cu")
+		(net "/5V")
+	)
+	(segment
+		(start 117.4 98.6)
+		(end 117.4 93.086016)
+		(width 1.5)
+		(layer "F.Cu")
+		(net "/5V")
+	)
+	(segment
+		(start 116 100)
+		(end 117.4 98.6)
+		(width 1.5)
+		(layer "F.Cu")
+		(net "/5V")
+	)
+	(segment
+		(start 113 121.2)
+		(end 116 118.2)
 		(width 1.5)
 		(layer "F.Cu")
@@
 		)
 		(min_thickness 0.25)
-		(fill
+		(fill yes
 			(thermal_gap 0.5)
 			(thermal_bridge_width 0.5)
